Commit message: urdf.xacro issues resolved

File: Kinematics/prac_urdf.urdf.xacro (robot description, xacro)
@@ -1,47 +1,47 @@
 <?xml version="1.0"?>
-<robto name="simple_robot">
-    <link name="base_link">
-        <visual>
-            <geometry>
-                <box size="0.5 0.3 0.1"/>
-            </geometry>
-            <material name="blue">
-                <color rgba="0 0 0 1"/>
-            </material>
-        </visual>
-        <collision>
-            <geometry>
-                <box size="0.5 0.3 0.1"/>
-            </geometry>
-        </collision>
-        <inertial>
-            <mass value="5.0"/>
-            <inertia ixx="0.01" ixy="0.0" ixz="0.0" iyy="0.01" iyz="0.0" izz="0.01"/>
-        </inertia>
-    </link>
-    <link name="wheel_link">
-        <visual>
-            <geometry>
-                <cylinder radius="0.1" length="0.05">
-            </geometry>
-            <material name="black">
-                <color rgba="0 0 0 1">
-            </material>
-        </visual>
-        <collision>
-            <geometry>
-                <cylinder raidus="0.1" length="0.05">
-            </geometry>
-        </collision>
-        <inertial>
-            <mass value="1.0">
-            <inertia ixx="0.001" ixy="0.0" ixz="0.0" iyy="0.001" iyz="0.0" izz="0.001"/>
-        </intertial>
-    </link>
-    <joint name="wheel_joint" type="continuous">
-        <parent link="wheel_base">
-        <child link="wheel_link">
-        <origin xyz="0.2 0.15 -0.05" rpy="0 0 0">
-        <axis xyz="0 1 0">
-    </joint>
+<robot name="simple_robot">
+  <link name="base_link">
+    <visual>
+      <geometry>
+        <box size="0.5 0.3 0.1"/>
+      </geometry>
+      <material name="blue">
+        <color rgba="0 0 0 1"/>
+      </material>
+    </visual>
+    <collision>
+      <geometry>
+        <box size="0.5 0.3 0.1"/>
+      </geometry>
+    </collision>
+    <inertial>
+      <mass value="5.0"/>
+      <inertia ixx="0.01" ixy="0.0" ixz="0.0" iyy="0.01" iyz="0.0" izz="0.01"/>
+    </inertial>
+  </link>
+  <link name="wheel_link">
+    <visual>
+      <geometry>
+        <cylinder radius="0.1" length="0.05"/>
+      </geometry>
+      <material name="black">
+        <color rgba="0 0 0 1"/>
+      </material>
+    </visual>
+    <collision>
+      <geometry>
+        <cylinder radius="0.1" length="0.05"/>
+      </geometry>
+    </collision>
+    <inertial>
+      <mass value="1.0"/>
+      <inertia ixx="0.001" ixy="0.0" ixz="0.0" iyy="0.001" iyz="0.0" izz="0.001"/>
+    </inertial>
+  </link>
+  <joint name="wheel_joint" type="continuous">
+    <parent link="base_link"/>
+    <child link="wheel_link"/>
+    <origin xyz="0.2 0.15 -0.05" rpy="0 0 0"/>
+    <axis xyz="0 1 0"/>
+  </joint>
 </robot>
